File: Half Bridge 1.kicad_sch (KiCad schematic)
At the start: 56 parts, among them J3 Conn_01x02_Pin, U1 M74VHC1GT86DFT1G, U2 ISG3204LA, U3 M74VHC1GT86DFT1G

Commit message: REV A
Parts:
- added TP5: TestPoint_Small, TestPoint:TestPoint_Pad_1.0x1.0mm, symbol Connector:TestPoint_Small
- TP3: renamed from TP1; footprint TestPoint:TestPoint_Pad_D1.0mm -> TestPoint:TestPoint_Pad_1.0x1.0mm
- TP4: renamed from TP2; footprint TestPoint:TestPoint_Pad_D1.0mm -> TestPoint:TestPoint_Pad_1.0x1.0mm
Connections:
- net OUT: now also TP5.1
