File: Power Stage.kicad_sch (KiCad schematic)
At the start: 5 parts, among them J1 Screw_Terminal_01x02, J2 Conn_01x02_Pin

Commit message: REV A
Parts:
- added TP1, TP2: TestPoint_Small, TestPoint:TestPoint_Pad_1.0x1.0mm, symbol Connector:TestPoint_Small
- gave numbers to parts that had none: 1
Connections:
- net +5V: now also TP1.1
- net GND: now also TP2.1
