File: Power Stage.kicad_pcb (KiCad board)
At the start: 4 copper layers, 50 x 50 mm, 125 parts, among them J1 Screw_Terminal_01x02, J2 Conn_01x02_Pin, J3 Conn_01x02_Pin, J4 Conn_01x02_Pin, J5 Screw_Terminal_01x04, U1 M74VHC1GT86DFT1G, U2 ISG3204LA, U3 M74VHC1GT86DFT1G, U4 M74VHC1GT86DFT1G, U5 ISG3204LA, U6 M74VHC1GT86DFT1G

Commit message: REV A
Parts:
- added ?: , , F.Cu at (109.9, 80.8)
- added ?: , , F.Cu at (140.0, 80.8)
- added C32: 10u, Capacitor_SMD:C_1210_3225Metric, F.Cu at (143.7, 86.6)
- added C32: 10u, Capacitor_SMD:C_1210_3225Metric, F.Cu at (106.2, 86.6)
- added J5: Conn_01x01_Pin, Connector_PinHeader_2.54mm:PinHeader_1x01_P2.54mm_Vertical, F.Cu at (103.5, 98.0)
- added J7: Conn_01x01_Pin, Connector_PinHeader_2.54mm:PinHeader_1x01_P2.54mm_Vertical, F.Cu at (146.5, 98.0)
- added TP1: TestPoint_Small, TestPoint:TestPoint_Pad_1.0x1.0mm, F.Cu at (104.6, 54.8)
- added TP10: TestPoint_Small, TestPoint:TestPoint_Pad_1.0x1.0mm, F.Cu at (146.6, 95.2)
- added TP2: TestPoint_Small, TestPoint:TestPoint_Pad_1.0x1.0mm, F.Cu at (102.0, 54.8)
- added TP5: TestPoint_Small, TestPoint:TestPoint_Pad_1.0x1.0mm, F.Cu at (123.0, 70.2)
- added TP8: TestPoint_Small, TestPoint:TestPoint_Pad_1.0x1.0mm, F.Cu at (127.0, 70.2)
- added TP9: TestPoint_Small, TestPoint:TestPoint_Pad_1.0x1.0mm, F.Cu at (103.5, 95.2)
- TP3: renamed from TP1; footprint TestPoint:TestPoint_Pad_D1.0mm -> TestPoint:TestPoint_Pad_1.0x1.0mm
- TP4: renamed from TP2; footprint TestPoint:TestPoint_Pad_D1.0mm -> TestPoint:TestPoint_Pad_1.0x1.0mm
- TP6: renamed from TP3; footprint TestPoint:TestPoint_Pad_D1.0mm -> TestPoint:TestPoint_Pad_1.0x1.0mm
- TP7: renamed from TP4; footprint TestPoint:TestPoint_Pad_D1.0mm -> TestPoint:TestPoint_Pad_1.0x1.0mm
- moved C89 21.7 mm to (140.0, 95.8), turned to 90 degrees
- moved C88 21.7 mm to (109.9, 95.8), turned to 90 degrees
- moved R17 11.6 mm to (103.0, 89.7), turned to 90 degrees
- moved R18 11.6 mm to (147.0, 89.7), turned to 90 degrees
- moved C90 9.10 mm to (103.0, 92.7), turned to 90 degrees
- moved C91 9.10 mm to (147.0, 92.7), turned to 90 degrees
- moved J2 1.90 mm to (104.6, 52.4), turned to -90 degrees
- moved C1 1.35 mm to (133.5, 83.2)
- moved C2 1.31 mm to (116.4, 83.2)
- moved J1 0.30 mm to (123.2, 53.3)
- moved J6 0.17 mm to (117.5, 95.2)
- renumbered J5 to J6
Routing:
- net +5V: track 0.00 -> 66.4 mm
- net Net-(J4-Pin_1): track 0.00 -> 11.9 mm
- net Net-(J3-Pin_1): track 0.00 -> 11.9 mm
- net VCC: track 0.00 -> 7.20 mm, vias 0 -> 97
- net Net-(U2-PWML): track 0.00 -> 6.61 mm
- net Net-(U5-PWML): track 0.00 -> 6.60 mm
- net Net-(U4-OUTY): track 0.00 -> 5.71 mm
- net Net-(U1-OUTY): track 0.00 -> 5.66 mm
- net GND: track 0.00 -> 3.43 mm, vias 0 -> 152
- net /Half Bridge 1/OUT: track 0.00 -> 2.75 mm
- net Net-(U2-HG): track 0.00 -> 2.73 mm
- net Net-(U5-LG): track 0.00 -> 2.70 mm
- net Net-(U2-LG): track 0.00 -> 2.70 mm
- net Net-(U5-HG): track 0.00 -> 2.70 mm
- net /Half Bridge 2/OUT: track 0.00 -> 2.68 mm
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- added copper zone on F.Cu, net +5V
- added copper zone on F.Cu, net /Half Bridge 1/OUT
- added copper zone on F.Cu, net /Half Bridge 2/OUT
- added copper zone on B.Cu, net GND
- added copper zone on F.Cu, net GND
- added copper zone on In1.Cu, net GND
- added copper zone on In2.Cu, net GND
- added copper zone on B.Cu, net Net-(C32-Pad2)
- added copper zone on B.Cu, net Net-(C34-Pad2)
- added copper zone on B.Cu, net Net-(C36-Pad2)
- added copper zone on B.Cu, net Net-(C38-Pad2)
- added copper zone on B.Cu, net Net-(C74-Pad2)
- added copper zone on B.Cu, net Net-(C76-Pad2)
- added copper zone on B.Cu, net Net-(C78-Pad2)
- added copper zone on B.Cu, net Net-(C80-Pad2)
- added copper zone on F.Cu, net Net-(J5-Pin_1)
- added copper zone on F.Cu, net Net-(J6-Pin_4)
- added copper zone on B.Cu, net VCC
- added copper zone on F.Cu, net VCC
Other:
- outline, holes or cut-outs redrawn
- board text added: "5V"
- board text added: "GND"
- board text added: "IN1"
- board text added: "IN2"
- board text added: "OUT1"
- board text added: "OUT2"
- board text added: "PWM1+"
- board text added: "PWM1-"
- board text added: "PWM2+"
- board text added: "PWM2-"
- board text added: "SW1"
- board text added: "SW2"
- board text added: "VCC"

Commit message: REV A1
Other:
- board text added: "REV A SALEM BEGIC"
Changed lines of the file:
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@@
+		)
+	)
+	(gr_text "REV A\nSALEM BEGIC\n"
+		(at 148.6 83.2 90)
+		(layer "F.SilkS" knockout)
+		(effects
+			(font
+				(size 1 1)
+				(thickness 0.2)
+				(bold yes)
+			)
+			(justify left bottom)
 		)
 	)
@@
 	)
 	(via
-		(at 148 81)
+		(at 149.1 80.7)
 		(size 0.6)
 		(drill 0.3)
@@
 	)
 	(via
-		(at 148 75)
-		(size 0.6)
-		(drill 0.3)
+		(at 149.1 74.7)
+		(size 0.6)
+		(drill 0.3)

Commit message: REV A2
Other:
- board text added: "POWER STAGE REV A SALEM BEGIC"
- board text removed: "REV A SALEM BEGIC"
Changed lines of the file:
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@@
 		)
 	)
-	(gr_text "REV A\nSALEM BEGIC\n"
-		(at 148.6 83.2 90)
+	(gr_text "POWER STAGE\nREV A\nSALEM BEGIC\n"
+		(at 149.4 83.2 90)
 		(layer "F.SilkS" knockout)
 		(effects
@@
 	)
 	(via
-		(at 149.1 80.7)
+		(at 148.1 83.5)
 		(size 0.6)
 		(drill 0.3)
@@
 	)
 	(via
-		(at 149.1 74.7)
-		(size 0.6)
-		(drill 0.3)
+		(at 148 72.4)
+		(size 0.6)
+		(drill 0.3)

Commit message: REV A3
Parts:
- added REF**: Fiducial_1mm_Mask2mm, Fiducial:Fiducial_1mm_Mask2mm, F.Cu at (102.4, 84.9)
- added REF**: Fiducial_1mm_Mask2mm, Fiducial:Fiducial_1mm_Mask2mm, F.Cu at (148.0, 53.0)
- added REF**: Fiducial_1mm_Mask2mm, Fiducial:Fiducial_1mm_Mask2mm, B.Cu at (148.0, 52.8)
- added REF**: Fiducial_1mm_Mask2mm, Fiducial:Fiducial_1mm_Mask2mm, B.Cu at (102.7, 94.9)
